File: kicad/ppg_pcb_v08.kicad_sch (KiCad schematic)
At the start: 37 parts, among them J1 12V, J2 GND, J3 TXP, J4 TXN, J5 RXP, J6 RXN, J7 SWDIO, J8 SWCLK, J9 NRST, U1 MAXM86161EFD+, U2 STM32C011F6U6, U3 XR33194, U4 MCP1703A-5002E/MC, U5 MCP1703A-3302E/MC, U6 XR33183

Commit message: Correct MCP1703A MC footprints and reroute RS-422 PCB
Parts:
- U2: footprint Package_DFN_QFN:ST_UFQFPN-20_3x3mm_P0.5mm -> SleepBud:ST_UFQFPN-20_3x3mm_P0.5mm_NoSilk
- U4, U5: footprint Package_DFN_QFN:DFN-8-1EP_2x3mm_P0.5mm_EP0.61x2.2mm -> SleepBud:MCP1703A_MC_DFN8_3x2mm_P0.5mm
Changed lines of the file:
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@@
   (text "VLDO bypass" (exclude_from_sim no) (at 60.96 150.495 0) (effects (font (size 1.27 1.27)) (justify left top)))
   (text "VREF bypass" (exclude_from_sim no) (at 93.98 150.495 0) (effects (font (size 1.27 1.27)) (justify left top)))
-  (symbol (lib_id "SleepBud:STM32C011F6U6") (at 208.28 83.82 0) (unit 1) (exclude_from_sim no) (in_bom yes) (on_board yes) (dnp no) (property "Reference" "U2" (at 177.8 41.91 0) (effects (font (size 1.27 1.27)) (justify left))) (property "Value" "STM32C011F6U6" (at 177.8 45.085 0) (effects (font (size 1.27 1.27)) (justify left))) (property "Footprint" "Package_DFN_QFN:ST_UFQFPN-20_3x3mm_P0.5mm" (at 208.28 83.82 0) (effects (font (size 1.27 1.27)) (hide yes))) (property "Datasheet" "" (at 208.28 83.82 0) (effects (font (size 1.27 1.27)) (hide yes))) (property "Description" "MCU, USART1 (PA9/PA10) <-> RS-422 driver/receiver, I2C1 (PB6/PB7) -> PPG; USART bootloader over the link" (at 208.28 83.82 0) (effects (font (size 1.27 1.27)) (hide yes))) (property "MPN" "" (at 208.28 83.82 0) (effects (font (size 1.27 1.27)) (hide yes))) (property "Manufacturer" "" (at 208.28 83.82 0) (effects (font (size 1.27 1.27)) (hide yes))) (pin "1") (pin "2") (pin "3") (pin "4") (pin "5") (pin "6") (pin "7") (pin "8") (pin "9") (pin "10") (pin "11") (pin "12") (pin "13") (pin "14") (pin "15") (pin "16") (pin "17") (pin "18") (pin "19") (pin "20") (instances (project "ppg_pcb_v08" (path "/49500282-0369-4cac-b640-45971f28f30c" (reference "U2") (unit 1)))))
+  (symbol (lib_id "SleepBud:STM32C011F6U6") (at 208.28 83.82 0) (unit 1) (exclude_from_sim no) (in_bom yes) (on_board yes) (dnp no) (property "Reference" "U2" (at 177.8 41.91 0) (effects (font (size 1.27 1.27)) (justify left))) (property "Value" "STM32C011F6U6" (at 177.8 45.085 0) (effects (font (size 1.27 1.27)) (justify left))) (property "Footprint" "SleepBud:ST_UFQFPN-20_3x3mm_P0.5mm_NoSilk" (at 208.28 83.82 0) (effects (font (size 1.27 1.27)) (hide yes))) (property "Datasheet" "" (at 208.28 83.82 0) (effects (font (size 1.27 1.27)) (hide yes))) (property "Description" "MCU, USART1 (PA9/PA10) <-> RS-422 driver/receiver, I2C1 (PB6/PB7) -> PPG; USART bootloader over the link" (at 208.28 83.82 0) (effects (font (size 1.27 1.27)) (hide yes))) (property "MPN" "" (at 208.28 83.82 0) (effects (font (size 1.27 1.27)) (hide yes))) (property "Manufacturer" "" (at 208.28 83.82 0) (effects (font (size 1.27 1.27)) (hide yes))) (pin "1") (pin "2") (pin "3") (pin "4") (pin "5") (pin "6") (pin "7") (pin "8") (pin "9") (pin "10") (pin "11") (pin "12") (pin "13") (pin "14") (pin "15") (pin "16") (pin "17") (pin "18") (pin "19") (pin "20") (instances (project "ppg_pcb_v08" (path "/49500282-0369-4cac-b640-45971f28f30c" (reference "U2") (unit 1)))))
   (wire (pts (xy 172.72 53.34) (xy 165.1 53.34)) (stroke (width 0) (type default)))
   (label "3V3" (at 165.1 53.34 180) (effects (font (size 1.27 1.27)) (justify right bottom)))
@@
   (wire (pts (xy 119.38 199.39) (xy 119.38 203.2)) (stroke (width 0) (type default)))
   (symbol (lib_id "SleepBud:GND") (at 119.38 203.2 0) (unit 1) (exclude_from_sim no) (in_bom no) (on_board yes) (dnp no) (property "Reference" "#PWR17" (at 119.38 203.2 0) (effects (font (size 1.27 1.27)) (hide yes))) (property "Value" "GND" (at 119.38 207.645 0) (effects (font (size 1.27 1.27)))) (property "Footprint" "" (at 119.38 203.2 0) (effects (font (size 1.27 1.27)) (hide yes))) (property "Datasheet" "" (at 119.38 203.2 0) (effects (font (size 1.27 1.27)) (hide yes))) (property "Description" "" (at 119.38 203.2 0) (effects (font (size 1.27 1.27)) (hide yes))) (pin "1") (instances (project "ppg_pcb_v08" (path "/49500282-0369-4cac-b640-45971f28f30c" (reference "#PWR17") (unit 1)))))
-  (symbol (lib_id "SleepBud:MCP1703A_DFN") (at 81.28 218.44 0) (unit 1) (exclude_from_sim no) (in_bom yes) (on_board yes) (dnp no) (property "Reference" "U4" (at 71.12 204.47 0) (effects (font (size 1.27 1.27)) (justify left))) (property "Value" "MCP1703A-5002E/MC" (at 71.12 207.645 0) (effects (font (size 1.27 1.27)) (justify left))) (property "Footprint" "Package_DFN_QFN:DFN-8-1EP_2x3mm_P0.5mm_EP0.61x2.2mm" (at 81.28 218.44 0) (effects (font (size 1.27 1.27)) (hide yes))) (property "Datasheet" "" (at 81.28 218.44 0) (effects (font (size 1.27 1.27)) (hide yes))) (property "Description" "LDO 12 V -> 5 V (VLED)" (at 81.28 218.44 0) (effects (font (size 1.27 1.27)) (hide yes))) (property "MPN" "" (at 81.28 218.44 0) (effects (font (size 1.27 1.27)) (hide yes))) (property "Manufacturer" "" (at 81.28 218.44 0) (effects (font (size 1.27 1.27)) (hide yes))) (pin "1") (pin "2") (pin "3") (pin "4") (pin "5") (pin "6") (pin "7") (pin "8") (pin "9") (instances (project "ppg_pcb_v08" (path "/49500282-0369-4cac-b640-45971f28f30c" (reference "U4") (unit 1)))))
+  (symbol (lib_id "SleepBud:MCP1703A_DFN") (at 81.28 218.44 0) (unit 1) (exclude_from_sim no) (in_bom yes) (on_board yes) (dnp no) (property "Reference" "U4" (at 71.12 204.47 0) (effects (font (size 1.27 1.27)) (justify left))) (property "Value" "MCP1703A-5002E/MC" (at 71.12 207.645 0) (effects (font (size 1.27 1.27)) (justify left))) (property "Footprint" "SleepBud:MCP1703A_MC_DFN8_3x2mm_P0.5mm" (at 81.28 218.44 0) (effects (font (size 1.27 1.27)) (hide yes))) (property "Datasheet" "${KIPRJMOD}/../datasheet/pdf/MCP1703A.pdf" (at 81.28 218.44 0) (effects (font (size 1.27 1.27)) (hide yes))) (property "Description" "LDO 12 V -> 5 V (VLED)" (at 81.28 218.44 0) (effects (font (size 1.27 1.27)) (hide yes))) (property "MPN" "" (at 81.28 218.44 0) (effects (font (size 1.27 1.27)) (hide yes))) (property "Manufacturer" "" (at 81.28 218.44 0) (effects (font (size 1.27 1.27)) (hide yes))) (pin "1") (pin "2") (pin "3") (pin "4") (pin "5") (pin "6") (pin "7") (pin "8") (pin "9") (instances (project "ppg_pcb_v08" (path "/49500282-0369-4cac-b640-45971f28f30c" (reference "U4") (unit 1)))))
   (wire (pts (xy 66.04 215.9) (xy 58.42 215.9)) (stroke (width 0) (type default)))
   (label "12V" (at 58.42 215.9 180) (effects (font (size 1.27 1.27)) (justify right bottom)))
@@
   (no_connect (at 83.82 231.14))
   (no_connect (at 86.36 231.14))
-  (symbol (lib_id "SleepBud:MCP1703A_DFN") (at 81.28 248.92 0) (unit 1) (exclude_from_sim no) (in_bom yes) (on_board yes) (dnp no) (property "Reference" "U5" (at 71.12 234.95 0) (effects (font (size 1.27 1.27)) (justify left))) (property "Value" "MCP1703A-3302E/MC" (at 71.12 238.125 0) (effects (font (size 1.27 1.27)) (justify left))) (property "Footprint" "Package_DFN_QFN:DFN-8-1EP_2x3mm_P0.5mm_EP0.61x2.2mm" (at 81.28 248.92 0) (effects (font (size 1.27 1.27)) (hide yes))) (property "Datasheet" "" (at 81.28 248.92 0) (effects (font (size 1.27 1.27)) (hide yes))) (property "Description" "LDO 5 V -> 3.3 V" (at 81.28 248.92 0) (effects (font (size 1.27 1.27)) (hide yes))) (property "MPN" "" (at 81.28 248.92 0) (effects (font (size 1.27 1.27)) (hide yes))) (property "Manufacturer" "" (at 81.28 248.92 0) (effects (font (size 1.27 1.27)) (hide yes))) (pin "1") (pin "2") (pin "3") (pin "4") (pin "5") (pin "6") (pin "7") (pin "8") (pin "9") (instances (project "ppg_pcb_v08" (path "/49500282-0369-4cac-b640-45971f28f30c" (reference "U5") (unit 1)))))
+  (symbol (lib_id "SleepBud:MCP1703A_DFN") (at 81.28 248.92 0) (unit 1) (exclude_from_sim no) (in_bom yes) (on_board yes) (dnp no) (property "Reference" "U5" (at 71.12 234.95 0) (effects (font (size 1.27 1.27)) (justify left))) (property "Value" "MCP1703A-3302E/MC" (at 71.12 238.125 0) (effects (font (size 1.27 1.27)) (justify left))) (property "Footprint" "SleepBud:MCP1703A_MC_DFN8_3x2mm_P0.5mm" (at 81.28 248.92 0) (effects (font (size 1.27 1.27)) (hide yes))) (property "Datasheet" "${KIPRJMOD}/../datasheet/pdf/MCP1703A.pdf" (at 81.28 248.92 0) (effects (font (size 1.27 1.27)) (hide yes))) (property "Description" "LDO 5 V -> 3.3 V" (at 81.28 248.92 0) (effects (font (size 1.27 1.27)) (hide yes))) (property "MPN" "" (at 81.28 248.92 0) (effects (font (size 1.27 1.27)) (hide yes))) (property "Manufacturer" "" (at 81.28 248.92 0) (effects (font (size 1.27 1.27)) (hide yes))) (pin "1") (pin "2") (pin "3") (pin "4") (pin "5") (pin "6") (pin "7") (pin "8") (pin "9") (instances (project "ppg_pcb_v08" (path "/49500282-0369-4cac-b640-45971f28f30c" (reference "U5") (unit 1)))))
   (wire (pts (xy 66.04 246.38) (xy 58.42 246.38)) (stroke (width 0) (type default)))
   (label "5V_LED" (at 58.42 246.38 180) (effects (font (size 1.27 1.27)) (justify right bottom)))
