File: kicad/ppg_pcb_v08.kicad_sch (KiCad schematic)
At the start: 37 parts, among them J1 12V, J2 GND, J3 TXP, J4 TXN, J5 RXP, J6 RXN, J7 SWDIO, J8 SWCLK, J9 NRST, U1 MAXM86161EFD+, U2 STM32C011F6U6, U3 XR33194, U4 MCP1703A-5002E/MC, U5 MCP1703A-3302E/MC, U6 XR33183

Commit message: Update PPG schematic with 0603 decoupling capacitors
Add C15/C16 100nF 16V X7R capacitors on 3V3 and include pending LDO_EN-to-PA7 and front SWD pad schematic changes. Preserve existing SWD ESD nets and symbol identities.

Publish generator dependencies, schematic previews, ERC results, and netlist verification. Native ERC reports zero violations; regenerated component data and all 123 numbered pin nets match.

PCB routing remains paused. PCB, project/rule files, BOM, and manufacturing outputs are intentionally excluded and remain unsynchronized with this schematic.
Parts:
- added C15, C16: 100nF 16V X7R, Capacitor_SMD:C_0201_0603Metric, symbol SleepBud:C
- added J10: GND, SleepBud:TestPad_D0.8_Front, symbol SleepBud:PAD
- added J11: 3V3_VTREF, SleepBud:TestPad_D0.8_Front, symbol SleepBud:PAD
- J7, J8, J9: footprint SleepBud:CablePad_D0.8 -> SleepBud:TestPad_D0.8_Front
Connections:
- net 3V3: now also C15.1, C16.1, J11.1; no longer U1.3 (LDO_EN)
- net GND: now also C15.2, C16.2, J10.1
- net LDO_EN: now reaches U2.12 (PA7)
- net LDO_EN: now also U1.3 (LDO_EN)
- no-connect marks 26 -> 25
Other:
- note added: "Additional 3V3 bypass / 0603 MLCC"
- moved on the sheet: J5, J6

Commit message: Save PPG routing, UART adapter, BOMs and 10-set panel
Record the current PPG schematic and routed six-layer PCB, UART adapter
with mounting holes, and default 0.25 mm via drill policy.

Include UART quantity BOMs in the requested PPG format and the validated
10-set PPG/UART panel Gerbers, drill files, placement coordinates and
review history. Preserve earlier manufacturing inputs and exclude local
backups, editor state and spreadsheet inspection caches.

Validation: current PPG/UART PCB hashes match the panel manifest; panel
ZIP CRC and checksums pass; 29 Python source files parse successfully.
Parts:
- added C17: 100 nF, Capacitor_SMD:C_0201_0603Metric, symbol SleepBud:C
- C1: value 10uF 6.3V X5R -> 10 µF; Dielectric (none) -> X5R; Voltage (none) -> 6.3 V
- C11, C6, C7: value 100nF -> 100 nF
- C12, C14, C4, C5: value 1uF 6.3V -> 1 µF; Voltage (none) -> 6.3 V
- C13: value 1uF 25V X7R -> 1 µF; Dielectric (none) -> X7R; Voltage (none) -> 25 V
- C15, C16: value 100nF 16V X7R -> 100 nF; Dielectric (none) -> X7R; Voltage (none) -> 16 V
- R1, R2: value 4.7k -> 4.7 kΩ
- R3: value 120/1% -> 120 Ω; Tolerance (none) -> 1%
- R4: value 10k -> 10 kΩ
- R5, R6, R7, R8: value 22 -> 22 Ω
- U3: value XR33194 -> XR33194ESBTR
- U6: value XR33183 -> XR33183ESBTR
Connections:
- net 5V_LED: now also C17.1
- net GND: now also C17.2
Other:
- note added: "R3: 120 Ω / 1% at the local RX cable pair."
- note added: "RS-422 bus TVS omitted; 22 Ω series retained. D1 protects supply, D6-D8 protect SWD. IEC immunity requires physical validation."
- note removed: "R3: 120/1% at the local RX cable pair."
- note removed: "RS-422 bus TVS omitted; 22 ohm series retained. D1 protects supply, D6-D8 protect SWD. IEC immunity requires physical validation."
- moved on the sheet: C1, C13, C14
