File: kicad/ppg_rs422_review.kicad_pcb (KiCad board)
At the start: 4 copper layers, 13.5 x 13.5 mm, 37 parts, among them J1 12V, J2 GND, J3 TXP, J4 TXN, J5 RXP, J6 RXN, J7 SWDIO, J8 SWCLK, J9 NRST, U1 MAXM86161EFD+, U2 STM32C011F6U6, U3 XR33194, U4 MCP1703A-5002E/MC, U5 MCP1703A-3302E/MC, U6 XR33183

Commit message: Save PPG routing, UART adapter, BOMs and 10-set panel
Record the current PPG schematic and routed six-layer PCB, UART adapter
with mounting holes, and default 0.25 mm via drill policy.

Include UART quantity BOMs in the requested PPG format and the validated
10-set PPG/UART panel Gerbers, drill files, placement coordinates and
review history. Preserve earlier manufacturing inputs and exclude local
backups, editor state and spreadsheet inspection caches.

Validation: current PPG/UART PCB hashes match the panel manifest; panel
ZIP CRC and checksums pass; 29 Python source files parse successfully.
Parts:
- C1: value 10uF 6.3V X5R -> 10 µF
- C11, C6, C7: value 100nF -> 100 nF
- C12, C14, C4, C5: value 1uF 6.3V -> 1 µF
- C13: value 1uF 25V X7R -> 1 µF
- R1, R2: value 4.7k -> 4.7 kΩ
- R3: value 120/1% -> 120 Ω
- R4: value 10k -> 10 kΩ
- R5, R6, R7, R8: value 22 -> 22 Ω
- U3: value XR33194 -> XR33194ESBTR
- U6: value XR33183 -> XR33183ESBTR
Changed lines of the file:
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@@
 			)
 		)
-		(property "Value" "1uF 6.3V"
+		(property "Value" "1 µF"
 			(at 0 -1.05 135)
 			(layer "B.Fab")
@@
 			)
 		)
-		(property "Value" "4.7k"
+		(property "Value" "4.7 kΩ"
 			(at 0 -1.05 0)
 			(layer "B.Fab")
@@
 			)
 		)
-		(property "Value" "100nF"
+		(property "Value" "100 nF"
 			(at 0 -1.05 135)
 			(layer "B.Fab")
@@
 			)
 		)
-		(property "Value" "22"
+		(property "Value" "22 Ω"
 			(at 0 -1.17 180)
 			(layer "B.Fab")
@@
 			)
 		)
-		(property "Value" "1uF 6.3V"
+		(property "Value" "1 µF"
 			(at 0 -1.05 315)
 			(layer "B.Fab")
@@
 			)
 		)
-		(property "Value" "1uF 25V X7R"
+		(property "Value" "1 µF"
 			(at 0 -1.16 90)
 			(layer "B.Fab")
@@
 			)
 		)
-		(property "Value" "10k"
+		(property "Value" "10 kΩ"
 			(at 0 -1.05 225)
 			(layer "B.Fab")
@@
 			)
 		)
-		(property "Value" "XR33194"
+		(property "Value" "XR33194ESBTR"
 			(at 0 -2.25 225)
 			(layer "B.Fab")
@@
 			)
 		)
-		(property "Value" "22"
+		(property "Value" "22 Ω"
 			(at 0 -1.17 0)
 			(layer "B.Fab")
@@
 			)
 		)
-		(property "Value" "22"
+		(property "Value" "22 Ω"
 			(at 0 -1.17 90)
 			(layer "B.Fab")
@@
 			)
 		)
-		(property "Value" "120/1%"
+		(property "Value" "120 Ω"
 			(at 0 -1.17 270)
 			(layer "B.Fab")
@@
 			)
 		)
-		(property "Value" "100nF"
+		(property "Value" "100 nF"
 			(at 0 -1.05 225)
 			(layer "B.Fab")
@@
 			)
 		)
-		(property "Value" "10uF 6.3V X5R"
+		(property "Value" "10 µF"
 			(at 0 -1.16 90)
 			(layer "B.Fab")
@@
 			)
 		)
-		(property "Value" "4.7k"
+		(property "Value" "4.7 kΩ"
 			(at 0 -1.05 0)
 			(layer "B.Fab")
@@
 			)
 		)
-		(property "Value" "1uF 6.3V"
+		(property "Value" "1 µF"
 			(at 0 -1.05 0)
 			(layer "B.Fab")
@@
 			)
 		)
-		(property "Value" "1uF 6.3V"
+		(property "Value" "1 µF"
 			(at 0 -1.05 0)
 			(layer "B.Fab")
@@
 			)
 		)
-		(property "Value" "XR33183"
+		(property "Value" "XR33183ESBTR"
 			(at 0 -2.25 0)
 			(layer "B.Fab")
@@
 			)
 		)
-		(property "Value" "100nF"
+		(property "Value" "100 nF"
 			(at 0 -1.05 90)
 			(layer "B.Fab")
@@
 			)
 		)
-		(property "Value" "22"
+		(property "Value" "22 Ω"
 			(at 0 -1.17 135)
 			(layer "B.Fab")
